Commit message: Add files via upload

File: URDF/Mk 3/urdf/CMU.urdf (robot description, URDF)
Before this commit: robot CMU, 13 links, 12 joints
Links:
- removed link L Feet
- removed link R Feet
- added link L Foot, mass 0.000518724222366595; collision mesh filename=package://CMU/meshes/L Foot.STL; visual mesh filename=package://CMU/meshes/L Foot.STL
- added link R Foot, mass 0.000518724222366593; collision mesh filename=package://CMU/meshes/R Foot.STL; visual mesh filename=package://CMU/meshes/R Foot.STL
Joints:
- removed joint L Feet
- removed joint R Feet
- added joint L Foot: type revolute, parent L Shin, child L Foot, origin xyz=0.03479 -0.0396 0 rpy=0 0 -0.0021136, axis 0 0 1, limit lower=0 upper=0 effort=0 velocity=0
- added joint R Foot: type revolute, parent R Shin, child R Foot, origin xyz=0.034784 -0.039603 0 rpy=0 0 0, axis 0 0 1, limit lower=0 upper=0 effort=0 velocity=0
- joint L Foreleg: axis 0 0 0 -> 1 0 0; origin xyz=0 -0.015891 -0.0084512 rpy=-0.14969 0 0 -> xyz=0 0.014316 0.010906 rpy=-3.1291 0 0
- joint L Hip 1: axis 0 0 1 -> 0 0 -1; origin xyz=-0.021005 0 0 rpy=1.5708 0 0 -> xyz=-0.021005 0 0 rpy=1.5708 0 3.1416
- joint L Hip 2: axis 0 0 0 -> 0 0 -1; origin xyz=0 -0.013139 0.007699 rpy=-1.5708 1.2153 3.1416 -> xyz=0 0 -0.0077 rpy=1.5708 0.35552 0
- joint L Shin: axis 0 0 0 -> 0 0 1
- joint L Thigh: axis 0 0 0 -> -1 0 0; origin xyz=0 0 0 rpy=-1.4086 0 1.5708 -> xyz=0 0 0.013141 rpy=1.5708 0 -3.1416
- joint R Foreleg: origin xyz=0 -0.0158930566714607 -0.00845048813014605 rpy=0 0 0 -> xyz=0 -0.015893 -0.0084505 rpy=0 0 0
- joint R Hip 1: origin xyz=0.0210048094716167 0 0 rpy=1.5707963267949 0 0 -> xyz=0.021005 0 0 rpy=1.5708 0 0
- joint R Hip 2: origin xyz=0 0 0.00769618467666837 rpy=1.5707963267949 1.31372099121825 0 -> xyz=0 0 0.0076962 rpy=1.5708 1.3137 0
- joint R Shin: origin xyz=0 -0.0535671183633322 0.0359517363775697 rpy=0 1.5707963267949 0 -> xyz=0 -0.053567 0.035952 rpy=0 1.5708 0
- joint R Thigh: origin xyz=0 0 0.0131387261681208 rpy=-1.5707963267949 0 1.5707963267949 -> xyz=0 0 0.013139 rpy=-1.5708 0 1.5708
