Commit message: Fixed Collision problem - added documentation

File: URDF/Mk 3/urdf/CMU3.urdf (robot description, URDF)
Before this commit: robot CMU, 13 links, 12 joints
Links:
- link base_link: geometry collision mesh filename=package://CMU/meshes/base_link_collision.STL; visual mesh filename=package://CMU/meshes/base_link.STL
