Commit message: URDF Mk 5 completed

File: URDF/Mk 4/urdf/CMU MK 4.urdf (robot description, URDF)
Before this commit: robot CMU MK 4, 19 links, 18 joints
Links:
- link L Foot: geometry collision mesh filename=package://CMU/meshes/L Foot.STL; visual mesh filename=package://CMU/meshes/L Foot.STL
- link L Foreleg: geometry collision mesh filename=package://CMU/meshes/L Foreleg.STL; visual mesh filename=package://CMU/meshes/L Foreleg.STL
- link L Hip 1: geometry collision mesh filename=package://CMU/meshes/L Hip 1.STL; visual mesh filename=package://CMU/meshes/L Hip 1.STL
- link L Hip 2: geometry collision mesh filename=package://CMU/meshes/L Hip 2.STL; visual mesh filename=package://CMU/meshes/L Hip 2.STL
- link L Shin: geometry collision mesh filename=package://CMU/meshes/L Shin.STL; visual mesh filename=package://CMU/meshes/L Shin.STL
- link L Thigh: geometry collision mesh filename=package://CMU/meshes/L Thigh.STL; visual mesh filename=package://CMU/meshes/L Thigh.STL
- link L_Linkage: geometry collision mesh filename=package://CMU/meshes/L_Linkage.STL; visual mesh filename=package://CMU/meshes/L_Linkage.STL
- link L_Servo: geometry collision mesh filename=package://CMU/meshes/L_Servo.STL; visual mesh filename=package://CMU/meshes/L_Servo.STL
- link L_Servo Joint: geometry collision mesh filename=package://CMU/meshes/L_Servo Joint.STL; visual mesh filename=package://CMU/meshes/L_Servo Joint.STL
- link R Foot: mass 0.00051872426680286 -> 0.000518724266802862; geometry collision mesh filename=package://CMU/meshes/R Foot.STL; visual mesh filename=package://CMU/meshes/R Foot.STL
- link R Foreleg: geometry collision mesh filename=package://CMU/meshes/R Foreleg.STL; visual mesh filename=package://CMU/meshes/R Foreleg.STL
- link R Hip 1: geometry collision mesh filename=package://CMU/meshes/R Hip 1.STL; visual mesh filename=package://CMU/meshes/R Hip 1.STL
- link R Hip 2: geometry collision mesh filename=package://CMU/meshes/R Hip 2.STL; visual mesh filename=package://CMU/meshes/R Hip 2.STL
- link R Shin: geometry collision mesh filename=package://CMU/meshes/R Shin.STL; visual mesh filename=package://CMU/meshes/R Shin.STL
- link R Thigh: geometry collision mesh filename=package://CMU/meshes/R Thigh.STL; visual mesh filename=package://CMU/meshes/R Thigh.STL
- link R_Linkage: geometry collision mesh filename=package://CMU/meshes/R_Linkage.STL; visual mesh filename=package://CMU/meshes/R_Linkage.STL
- link R_Servo: geometry collision mesh filename=package://CMU/meshes/R_Servo.STL; visual mesh filename=package://CMU/meshes/R_Servo.STL
- link R_Servo Joint: mass 5.90677466361002E-05 -> 5.90677466361003E-05; geometry collision mesh filename=package://CMU/meshes/R_Servo Joint.STL; visual mesh filename=package://CMU/meshes/R_Servo Joint.STL
- link base_link: geometry collision mesh filename=package://CMU/meshes/base_link_collision.STL; visual mesh filename=package://CMU/meshes/base_link.STL
Joints:
- joint L Hip 2: axis 0 0 0 -> 0 0 1
- joint L Thigh: axis 0 0 0 -> -1 0 0

File: URDF/Mk 5/urdf/CMU Mk 5.urdf (robot description, URDF)
Before this commit: robot CMU MK 4, 19 links, 18 joints
Links:
- removed link L Foot
- removed link L Foreleg
- removed link L Hip 1
- removed link L Hip 2
- removed link L Shin
- removed link L Thigh
- removed link L_Servo Joint
- removed link R Foot
- removed link R Foreleg
- removed link R Hip 1
- removed link R Hip 2
- removed link R Shin
- removed link R Thigh
- removed link R_Servo Joint
- added link L_Foot, mass 0.00051872433253689; collision mesh filename=package://CMU Mk 5/meshes/L_Foot.STL; visual mesh filename=package://CMU Mk 5/meshes/L_Foot.STL
- added link L_Foreleg, mass 0.00244939435652077; collision mesh filename=package://CMU Mk 5/meshes/L_Foreleg.STL; visual mesh filename=package://CMU Mk 5/meshes/L_Foreleg.STL
- added link L_Hip_1, mass 0.000490672959387971; collision mesh filename=package://CMU Mk 5/meshes/L_Hip_1.STL; visual mesh filename=package://CMU Mk 5/meshes/L_Hip_1.STL
- added link L_Hip_2, mass 0.00100456223004492; collision mesh filename=package://CMU Mk 5/meshes/L_Hip_2.STL; visual mesh filename=package://CMU Mk 5/meshes/L_Hip_2.STL
- added link L_Servo_Link, mass 5.90677466361003E-05; collision mesh filename=package://CMU Mk 5/meshes/L_Servo_Link.STL; visual mesh filename=package://CMU Mk 5/meshes/L_Servo_Link.STL
- added link L_Shin, mass 0.00129204638168326; collision mesh filename=package://CMU Mk 5/meshes/L_Shin.STL; visual mesh filename=package://CMU Mk 5/meshes/L_Shin.STL
- added link L_Thigh, mass 0.00259524215854131; collision mesh filename=package://CMU Mk 5/meshes/L_Thigh.STL; visual mesh filename=package://CMU Mk 5/meshes/L_Thigh.STL
- added link R_Foot, mass 0.000518724266802862; collision mesh filename=package://CMU Mk 5/meshes/R_Foot.STL; visual mesh filename=package://CMU Mk 5/meshes/R_Foot.STL
- added link R_Foreleg, mass 0.00244939435652077; collision mesh filename=package://CMU Mk 5/meshes/R_Foreleg.STL; visual mesh filename=package://CMU Mk 5/meshes/R_Foreleg.STL
- added link R_Hip_1, mass 0.00049067295938797; collision mesh filename=package://CMU Mk 5/meshes/R_Hip_1.STL; visual mesh filename=package://CMU Mk 5/meshes/R_Hip_1.STL
- added link R_Hip_2, mass 0.00100456223004492; collision mesh filename=package://CMU Mk 5/meshes/R_Hip_2.STL; visual mesh filename=package://CMU Mk 5/meshes/R_Hip_2.STL
- added link R_Servo_Link, mass 5.90677466361003E-05; collision mesh filename=package://CMU Mk 5/meshes/R_Servo_Link.STL; visual mesh filename=package://CMU Mk 5/meshes/R_Servo_Link.STL
- added link R_Shin, mass 0.00129204638168326; collision mesh filename=package://CMU Mk 5/meshes/R_Shin.STL; visual mesh filename=package://CMU Mk 5/meshes/R_Shin.STL
- added link R_Thigh, mass 0.00259524215854131; collision mesh filename=package://CMU Mk 5/meshes/R_Thigh.STL; visual mesh filename=package://CMU Mk 5/meshes/R_Thigh.STL
- link L_Linkage: geometry collision mesh filename=package://CMU Mk 5/meshes/L_Linkage.STL; visual mesh filename=package://CMU Mk 5/meshes/L_Linkage.STL
- link L_Servo: geometry collision mesh filename=package://CMU Mk 5/meshes/L_Servo.STL; visual mesh filename=package://CMU Mk 5/meshes/L_Servo.STL
- link R_Linkage: geometry collision mesh filename=package://CMU Mk 5/meshes/R_Linkage.STL; visual mesh filename=package://CMU Mk 5/meshes/R_Linkage.STL
- link R_Servo: geometry collision mesh filename=package://CMU Mk 5/meshes/R_Servo.STL; visual mesh filename=package://CMU Mk 5/meshes/R_Servo.STL
- link base_link: geometry collision mesh filename=package://CMU Mk 5/meshes/base_link_collision.STL; visual mesh filename=package://CMU Mk 5/meshes/base_link.STL
Joints:
- removed joint L Foot
- removed joint L Foreleg
- removed joint L Hip 1
- removed joint L Hip 2
- removed joint L Shin
- removed joint L Thigh
- removed joint L_Servo Joint
- removed joint R Foot
- removed joint R Foreleg
- removed joint R Hip 1
- removed joint R Hip 2
- removed joint R Shin
- removed joint R Thigh
- removed joint R_Servo Joint
- added joint L_Foot: type revolute, parent L_Shin, child L_Foot, origin xyz=0 0.050359 -0.015576 rpy=0 -1.3777 -1.5708, axis 0 -1 0, limit lower=0 upper=0 effort=0 velocity=0
- added joint L_Foreleg: type revolute, parent L_Thigh, child L_Foreleg, origin xyz=0 -0.015892 -0.0084481 rpy=-1.4674 0 0, axis -1 0 0, limit lower=0 upper=0 effort=0 velocity=0
- added joint L_Hip_1: type revolute, parent base_link, child L_Hip_1, origin xyz=-0.021005 0 0 rpy=1.5708 0 0, axis 0 0 1, limit lower=0 upper=0 effort=0 velocity=0
- added joint L_Hip_2: type revolute, parent L_Hip_1, child L_Hip_2, origin xyz=0 -0.013139 0.0076997 rpy=-1.5708 1.3223 3.1416, axis 0 0 1, limit lower=0 upper=0 effort=0 velocity=0
- added joint L_Servo_Link: type revolute, parent L_Servo, child L_Servo_Link, origin xyz=0 -0.0075599 0 rpy=-1.8217 0 -3.1416, axis -1 0 0, limit lower=0 upper=0 effort=0 velocity=0
- added joint L_Shin: type revolute, parent L_Foreleg, child L_Shin, origin xyz=0 0.064515 0 rpy=-1.1349 0 0, axis -1 0 0, limit lower=0 upper=0 effort=0 velocity=0
- added joint L_Thigh: type revolute, parent L_Hip_2, child L_Thigh, origin xyz=0 0 0 rpy=-2.4963 0 -1.5708, axis -1 0 0, limit lower=0 upper=0 effort=0 velocity=0
- added joint R_Foot: type revolute, parent R_Shin, child R_Foot, origin xyz=0 0.050358 -0.015576 rpy=1.4972 0 0, axis -1 0 0, limit lower=0 upper=0 effort=0 velocity=0
- added joint R_Foreleg: type revolute, parent R_Thigh, child R_Foreleg, origin xyz=0 0.018 0 rpy=-2.0409 0 3.1416, axis -1 0 0, limit lower=0 upper=0 effort=0 velocity=0
- added joint R_Hip_1: type revolute, parent base_link, child R_Hip_1, origin xyz=0.021005 0 0 rpy=1.5708 -0.062045 0, axis 0 0 1, limit lower=0 upper=0 effort=0 velocity=0
- added joint R_Hip_2: type revolute, parent R_Hip_1, child R_Hip_2, origin xyz=0 0 0.0076962 rpy=1.5708 1.45 0, axis 0 0 1, limit lower=0 upper=0 effort=0 velocity=0
- added joint R_Servo_Link: type revolute, parent R_Servo, child R_Servo_Link, origin xyz=0.0075599 0 0 rpy=-1.5864 0 -1.5708, axis -1 0 0, limit lower=0 upper=0 effort=0 velocity=0
- added joint R_Shin: type revolute, parent R_Foreleg, child R_Shin, origin xyz=0 0.064516 0 rpy=-1.0363 0 0, axis -1 0 0, limit lower=0 upper=0 effort=0 velocity=0
- added joint R_Thigh: type revolute, parent R_Hip_2, child R_Thigh, origin xyz=0 0 0.013139 rpy=1.9476 0 1.5708, axis -1 0 0, limit lower=0 upper=0 effort=0 velocity=0
- joint L_Linkage: parent L Thigh -> L_Thigh
- joint L_Servo: parent L Shin -> L_Shin
- joint R_Linkage: parent R Thigh -> R_Thigh
- joint R_Servo: parent R Shin -> R_Shin
